File: eagle/bp/js220_bp.brd (EAGLE design)
At the start: 95 x 24.7 mm, 2 parts

Commit message: Updated for JS220 p3.
Parts:
- removed H3: HOLE_#6_NORESTRICT, jetperch:HOLE_3.5MM_NORESTRICT
- added H1: HOLE_#6_NORESTRICT, jetperch:HOLE_3.5MM_NORESTRICT
- moved H2 87.4 mm to (91.2, 12.3)
Other:
- board text added: "Controller Status"
- board text added: "GPIO and trigger are referenced to USB ground"
- board text added: "JS220_ep_pcb_revB JS220 End Panel, Rev B 2022 Jetperch LLC"
- board text added: "OUT0 GND IN2 IN0 Vref"
- board text added: "OUT1 GND IN3 IN1 GND"
- board text added: "Place all markings on back (including pcb order number). Add flammability rating marking on back, such as 94V-0. The front-side surface is cosmetic - reject units with scratches and blemishes."
- board text added: "Trigger"
- board text removed: "GND IN1 IN3 GND OUT1"
- board text removed: "JS220 Back Panel Rev B 2022 Jetperch LLC"
- board text removed: "Status"
- board text removed: "To host computer"
- board text removed: "Trigger In/Out"
- board text removed: "Vref IN0 IN2 GND OUT0"
Changed lines of the file:
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@@
 <drawing>
 <settings>
-<setting alwaysvectorfont="no"/>
+<setting alwaysvectorfont="yes"/>
 <setting verticaltext="up"/>
 </settings>
@@
 <board>
 <plain>
-<text x="47.5" y="20.2" size="1.27" layer="26" font="vector" ratio="20" rot="MR0" align="center">JS220 Back Panel
-Rev B
+<text x="47.5" y="20.2" size="1.27" layer="26" font="vector" ratio="20" rot="MR0" align="center">JS220_ep_pcb_revB
+JS220 End Panel, Rev B
 2022 Jetperch LLC</text>
 <dimension x1="0" y1="12.35" x2="95" y2="12.35" x3="47.5" y3="40.64" textsize="1.778" layer="47" dtype="horizontal"/>
@@
 <wire x1="82.65" y1="24.7" x2="12.35" y2="24.7" width="0" layer="20"/>
 <wire x1="12.35" y1="24.7" x2="0" y2="12.35" width="0" layer="20" curve="90"/>
-<text x="38.75" y="20" size="1.5" layer="29" font="vector" ratio="20" align="center">Status</text>
+<text x="38.75" y="17" size="1.27" layer="29" font="vector" ratio="20" align="center">Controller
+Status</text>
 <hole x="38.75" y="12.5" drill="3.3"/>
 <wire x1="74" y1="8.68" x2="92" y2="8.68" width="0.254" layer="22"/>
@@
 <wire x1="69.12" y1="5.645" x2="66.32" y2="5.645" width="0" layer="20"/>
 <wire x1="66.32" y1="5.645" x2="66.32" y2="17.465" width="0" layer="20"/>
-<text x="47.5" y="20" size="1.5" layer="29" font="vector" ratio="20" align="center">USB</text>
-<text x="67.72" y="20" size="1.5" layer="29" font="vector" ratio="20" align="center">Trigger
-In/Out</text>
-<text x="67.72" y="2" size="1" layer="29" font="vector" ratio="20" align="bottom-center">Out: 3.3V, 50 Ω
+<text x="47.5" y="13.6" size="2" layer="29" font="vector" ratio="20" align="center">USB</text>
+<text x="67.72" y="19.6" size="2" layer="29" font="vector" ratio="20" align="center">Trigger</text>
+<text x="67.72" y="3.5" size="1" layer="29" font="vector" ratio="20" distance="40" align="center">Out: 3.3V, 50 Ω
 In: TTL &amp; 3.3V compatible</text>
-<text x="47.5" y="2" size="1" layer="29" font="vector" ratio="20" align="bottom-center">To host computer
-</text>
+<text x="47.5" y="3.5" size="1" layer="29" font="vector" ratio="20" align="center">GPIO and trigger are
+referenced to USB ground</text>
 <wire x1="20.23" y1="9.58" x2="34.33" y2="9.58" width="0" layer="20"/>
 <wire x1="34.33" y1="9.58" x2="34.33" y2="16.58" width="0" layer="20"/>
@@
 <wire x1="24.53" y1="16.58" x2="20.23" y2="16.58" width="0" layer="20"/>
 <wire x1="20.23" y1="16.58" x2="20.23" y2="9.58" width="0" layer="20"/>
-<text x="27.28" y="3.49" size="1.5" layer="29" font="vector" ratio="20" align="center">GPIO</text>
-<text x="27.28" y="8.98" size="1.27" layer="29" font="vector" ratio="20" distance="100" rot="R90" align="center-right">GND
+<text x="27.28" y="3.5" size="2" layer="29" font="vector" ratio="20" align="center">GPIO</text>
+<text x="27.28" y="8.98" size="1.27" layer="29" font="vector" ratio="20" distance="100" rot="SR270" align="center-left">OUT1
+GND
+IN3
 IN1
-IN3
+GND</text>
+<text x="27.28" y="18.54" size="1.27" layer="29" font="vector" ratio="20" distance="100" rot="SR270" align="center-right">OUT0
 GND
-OUT1</text>
-<text x="27.28" y="18.54" size="1.27" layer="29" font="vector" ratio="20" distance="100" rot="R90" align="center-left">Vref
+IN2
 IN0
-IN2
-GND
-OUT0</text>
+Vref</text>
+<text x="17.573" y="-22.892" size="1.778" layer="153">Place all markings on back (including pcb order number).
+Add flammability rating marking on back, such as 94V-0.
+The front-side surface is cosmetic - reject units with scratches and blemishes.</text>
 </plain>
 <attributes>
@@
 </autorouter>
 <elements>
-<element name="H2" library="jetperch" package="HOLE_3.5MM_NORESTRICT" value="HOLE_#6_NORESTRICT" x="3.79" y="12.35" smashed="yes"/>
-<element name="H3" library="jetperch" package="HOLE_3.5MM_NORESTRICT" value="HOLE_#6_NORESTRICT" x="91.21" y="12.35" smashed="yes"/>
+<element name="H1" library="jetperch" package="HOLE_3.5MM_NORESTRICT" value="HOLE_#6_NORESTRICT" x="3.79" y="12.35" smashed="yes">
+<attribute name="POPULATE" value="0" x="3.79" y="12.35" size="1.778" layer="27" display="off"/>
+</element>
+<element name="H2" library="jetperch" package="HOLE_3.5MM_NORESTRICT" value="HOLE_#6_NORESTRICT" x="91.21" y="12.35" smashed="yes">
+<attribute name="POPULATE" value="0" x="91.21" y="12.35" size="1.778" layer="27" display="off"/>
+</element>
 </elements>
 <signals>

Commit message: Updated for beta build.
Other:
- outline, holes or cut-outs redrawn
- board text added: "js220_ep_pcb_revC JS220 End Panel, Rev C 2022 Jetperch LLC"
- board text removed: "JS220_ep_pcb_revB JS220 End Panel, Rev B 2022 Jetperch LLC"
Changed lines of the file:
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@@
 <drawing>
 <settings>
-<setting alwaysvectorfont="yes"/>
+<setting alwaysvectorfont="no"/>
 <setting verticaltext="up"/>
 </settings>
@@
 <board>
 <plain>
-<text x="47.5" y="20.2" size="1.27" layer="26" font="vector" ratio="20" rot="MR0" align="center">JS220_ep_pcb_revB
-JS220 End Panel, Rev B
+<text x="47.5" y="20.2" size="1.27" layer="26" font="vector" ratio="20" rot="MR0" align="center">js220_ep_pcb_revC
+JS220 End Panel, Rev C
 2022 Jetperch LLC</text>
 <dimension x1="0" y1="12.35" x2="95" y2="12.35" x3="47.5" y3="40.64" textsize="1.778" layer="47" dtype="horizontal"/>
@@
 <vertex x="47.5" y="1.25"/>
 </polygon>
-<hole x="67.72" y="11.555" drill="10.45"/>
-<wire x1="52" y1="9.58" x2="52" y2="9.89" width="0" layer="20"/>
-<wire x1="52" y1="9.89" x2="50.6" y2="11.29" width="0" layer="20" curve="90"/>
-<wire x1="50.6" y1="11.29" x2="44.4" y2="11.29" width="0" layer="20"/>
-<wire x1="44.4" y1="11.29" x2="43" y2="9.89" width="0" layer="20" curve="90"/>
-<wire x1="43" y1="9.89" x2="43" y2="9.58" width="0" layer="20"/>
-<wire x1="43" y1="9.58" x2="44.4" y2="8.18" width="0" layer="20" curve="90"/>
-<wire x1="44.4" y1="8.18" x2="50.6" y2="8.18" width="0" layer="20"/>
-<wire x1="50.6" y1="8.18" x2="52" y2="9.58" width="0" layer="20" curve="90"/>
-<wire x1="66.32" y1="17.465" x2="69.12" y2="17.465" width="0" layer="20"/>
-<wire x1="69.12" y1="17.465" x2="69.12" y2="5.645" width="0" layer="20"/>
-<wire x1="69.12" y1="5.645" x2="66.32" y2="5.645" width="0" layer="20"/>
-<wire x1="66.32" y1="5.645" x2="66.32" y2="17.465" width="0" layer="20"/>
+<hole x="67.72" y="12.355" drill="10.05"/>
+<wire x1="42.85" y1="9.785" x2="44.505" y2="8.13" width="0" layer="20" curve="90"/>
+<wire x1="44.505" y1="8.13" x2="50.495" y2="8.13" width="0" layer="20"/>
+<wire x1="50.495" y1="8.13" x2="52.15" y2="9.785" width="0" layer="20" curve="90"/>
+<wire x1="52.15" y1="9.785" x2="50.495" y2="11.44" width="0" layer="20" curve="90"/>
+<wire x1="50.495" y1="11.44" x2="44.505" y2="11.44" width="0" layer="20"/>
+<wire x1="44.505" y1="11.44" x2="42.85" y2="9.785" width="0" layer="20" curve="90"/>
+<wire x1="66.52" y1="18.065" x2="68.92" y2="18.065" width="0" layer="20"/>
+<wire x1="68.92" y1="18.065" x2="68.92" y2="6.645" width="0" layer="20"/>
+<wire x1="68.92" y1="6.645" x2="66.52" y2="6.645" width="0" layer="20"/>
+<wire x1="66.52" y1="6.645" x2="66.52" y2="18.065" width="0" layer="20"/>
 <text x="47.5" y="13.6" size="2" layer="29" font="vector" ratio="20" align="center">USB</text>
 <text x="67.72" y="19.6" size="2" layer="29" font="vector" ratio="20" align="center">Trigger</text>
