File: eagle/bp/js220_bp.sch (EAGLE design)
At the start: 2 parts

Commit message: Updated for JS220 p3.
Parts:
- removed H3: HOLE_#6_NORESTRICT, jetperch:HOLE_#6_NORESTRICT
- added H1: HOLE_#6_NORESTRICT, jetperch:HOLE_#6_NORESTRICT
- H2: POPULATE (none) -> 0
Changed lines of the file:
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@@
 <parts>
 <part name="FRAME1" library="frames" library_urn="urn:adsk.eagle:library:229" deviceset="FRAME_A_L" device="" value="PG1"/>
-<part name="H2" library="jetperch" deviceset="HOLE" device="_#6_NORESTRICT" value="HOLE_#6_NORESTRICT"/>
-<part name="H3" library="jetperch" deviceset="HOLE" device="_#6_NORESTRICT" value="HOLE_#6_NORESTRICT"/>
+<part name="H1" library="jetperch" deviceset="HOLE" device="_#6_NORESTRICT" value="HOLE_#6_NORESTRICT">
+<attribute name="POPULATE" value="0"/>
+</part>
+<part name="H2" library="jetperch" deviceset="HOLE" device="_#6_NORESTRICT" value="HOLE_#6_NORESTRICT">
+<attribute name="POPULATE" value="0"/>
+</part>
+<part name="PCB1" library="jetperch" deviceset="PCB" device="" value="JS220_ep_pcb_revB">
+<attribute name="MPN" value="JS220_fp_bp_pcb_revB"/>
+<attribute name="POPULATE" value="1"/>
+</part>
 </parts>
 <sheets>
@@
 <attribute name="DRAWING_NAME" x="190.5" y="19.05" size="2.54" layer="94"/>
 </instance>
-<instance part="H2" gate="G$1" x="7.62" y="200.66" smashed="yes"/>
-<instance part="H3" gate="G$1" x="12.7" y="200.66" smashed="yes"/>
+<instance part="H1" gate="G$1" x="7.62" y="200.66" smashed="yes">
+<attribute name="POPULATE" x="7.62" y="200.66" size="1.778" layer="96" display="off"/>
+</instance>
+<instance part="H2" gate="G$1" x="12.7" y="200.66" smashed="yes">
+<attribute name="POPULATE" x="12.7" y="200.66" size="1.778" layer="96" display="off"/>
+</instance>
+<instance part="PCB1" gate="G$1" x="12.7" y="190.5" smashed="yes">
+<attribute name="VALUE" x="7.62" y="185.42" size="1.27" layer="96"/>
+<attribute name="NAME" x="7.62" y="193.548" size="1.27" layer="95"/>
+<attribute name="POPULATE" x="12.7" y="190.5" size="1.27" layer="96" display="off"/>
+<attribute name="MPN" x="12.7" y="190.5" size="1.27" layer="96" display="off"/>
+</instance>
 </instances>
 <busses>

Commit message: Updated for beta build.
Other:
- note added: "C"
- note removed: "B"
Changed lines of the file:
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@@
 <attribute name="POPULATE" value="0"/>
 </part>
-<part name="PCB1" library="jetperch" deviceset="PCB" device="" value="JS220_ep_pcb_revB">
-<attribute name="MPN" value="JS220_fp_bp_pcb_revB"/>
+<part name="PCB1" library="jetperch" deviceset="PCB" device="" value="JS220_ep_pcb_revC">
 <attribute name="POPULATE" value="1"/>
 </part>
@@
 <plain>
 <text x="177.8" y="26.162" size="5.08" layer="97">Back Panel</text>
-<text x="266.7" y="6.35" size="3.175" layer="97">B</text>
+<text x="266.7" y="6.35" size="3.175" layer="97">C</text>
 </plain>
 <instances>
@@
 <attribute name="NAME" x="7.62" y="193.548" size="1.27" layer="95"/>
 <attribute name="POPULATE" x="12.7" y="190.5" size="1.27" layer="96" display="off"/>
-<attribute name="MPN" x="12.7" y="190.5" size="1.27" layer="96" display="off"/>
 </instance>
 </instances>
