File: eagle/fp_binding_posts/js220_fp_binding_posts.brd (EAGLE design)
At the start: 95 x 24.7 mm, 9 parts, among them J1 111-0703-001, J2 111-0702-001, J4 111-0702-001, J5 TSM-105-01-S-SV

Commit message: Updated for p3
Parts:
- added J3: 111-0702-001, jetperch:BINDING_POST_6
- J4: value 111-0702-001 -> 111-0707-001
- J5: value TSM-105-01-S-SV -> TSM-105-01-L-SV-A; device jetperch:CONN_0.1_5X1_MSA -> jetperch:CONN_0.1_3X2_MSA
- moved J4 19.1 mm to (76.1, 12.3)
- moved J5 5.36 mm to (47.5, 11.1)
Connections:
- removed net EXT_IN: J2.1, J5.01, J5.02
- removed net EXT_NEG: J1.1, J5.03
- removed net EXT_OUT: J4.1, J5.04, J5.05
- new net I+: J3.1, J5.1, J5.2
- new net I-: J4.1, J5.3, J5.4
- new net V+: J2.1, J5.6
- new net V-: J1.1, J5.5
Routing:
- net I-: track 0.00 -> 70.7 mm
- net EXT_NEG: track 44.6 -> 0.00 mm
- net V-: track 0.00 -> 32.5 mm
- net I+: track 0.00 -> 16.1 mm
- net V+: track 0.00 -> 7.50 mm
- added copper zone on layer 16, net I+
- added copper zone on layer 16, net I-
- removed copper zone on layer 16, net EXT_IN
- removed copper zone on layer 16, net EXT_OUT
Other:
- outline, holes or cut-outs redrawn
- board text added: "Install J1-J4 on other side"
- board text added: "Isolated ±48V max to USB ground"
- board text added: "J1 Black"
- board text added: "J2 Red"
- board text added: "J3 Red"
- board text added: "J4 Yellow"
- board text added: "JS220 Binding Post Front Panel Rev C 2022 Jetperch LLC"
- board text added: "±15V"
- board text added: "±3A"
- board text removed: "Black"
- board text removed: "Gnd In1 In3 Out1"
- board text removed: "JS220 Binding Post Front Panel Rev A 2021 Jetperch LLC"
- board text removed: "Red"
- board text removed: "Vref In0 In2 Out0"
- board text removed: "Yellow"

Commit message: Updated to rev B.
Other:
- board text added: "Install J1-J4 with nut on this side"
- board text added: "JS220 Binding Post Front Panel Rev B 2022 Jetperch LLC"
- board text removed: "Install J1-J4 on other side"
- board text removed: "JS220 Binding Post Front Panel Rev C 2022 Jetperch LLC"
Changed lines of the file:
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@@
 +    -</text>
 <text x="47.5" y="20.2" size="1.27" layer="26" font="vector" ratio="20" rot="MR0" align="center">JS220 Binding Post Front Panel
-Rev C
+Rev B
 2022 Jetperch LLC</text>
 <dimension x1="0" y1="12.35" x2="95" y2="12.35" x3="47.5" y3="40.64" textsize="1.778" layer="47" dtype="horizontal"/>
@@
 Red</text>
 <wire x1="80" y1="8.68" x2="92" y2="8.68" width="0.254" layer="22"/>
-<text x="47.5" y="2.2" size="1.27" layer="26" font="vector" ratio="20" rot="MR0" align="center">Install J1-J4 on other side</text>
+<text x="47.5" y="2.2" size="1.27" layer="26" font="vector" ratio="20" rot="MR0" align="center">Install J1-J4 with nut on this side</text>
 <text x="28.45" y="17.6022" size="1.27" layer="29" font="vector" ratio="20" distance="25" align="center">±15V</text>
 <text x="47.5" y="3.2512" size="1.27" layer="29" font="vector" ratio="20" distance="25" align="center">Isolated

Commit message: Updated for JS220 p3.
Parts:
- removed H3: HOLE_#6_NORESTRICT, jetperch:HOLE_3.5MM_NORESTRICT
- added H1: HOLE_#6_NORESTRICT, jetperch:HOLE_3.5MM_NORESTRICT
- moved H2 87.4 mm to (91.2, 12.3)
Other:
- board text added: "+"
- board text added: "-"
- board text added: "2x holes 4x connectors"
- board text added: "Current"
- board text added: "JS220_fp_bp_pcb_revB JS220 Binding Post Front Panel, Rev B 2022 Jetperch LLC"
- board text added: "Place all markings on back (including pcb order number). Add flammability rating marking on back, such as 94V-0. The front-side surface is cosmetic - reject units with scratches and blemishes."
- board text added: "Sensor Status"
- board text added: "Voltage"
- board text added: "±10A pulse"
- board text removed: "Current + -"
- board text removed: "JS220 Binding Post Front Panel Rev B 2022 Jetperch LLC"
- board text removed: "Status"
- board text removed: "Voltage - +"
Changed lines of the file:
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@@
 <setting verticaltext="up"/>
 </settings>
-<grid distance="5" unitdist="mil" unit="mil" style="lines" multiple="1" display="no" altdistance="0.1" altunitdist="mm" altunit="mm"/>
+<grid distance="1" unitdist="mm" unit="mm" style="lines" multiple="1" display="no" altdistance="0.1" altunitdist="mm" altunit="mm"/>
 <layers>
 <layer number="1" name="Top" color="4" fill="1" visible="yes" active="yes"/>
@@
 <board>
 <plain>
-<text x="28.45" y="18.5" size="3" layer="29" font="vector" ratio="20" distance="40" align="center">Voltage
--    +</text>
-<text x="66.55" y="18.5" size="3" layer="29" font="vector" ratio="20" distance="40" align="center">Current
-+    -</text>
-<text x="47.5" y="20.2" size="1.27" layer="26" font="vector" ratio="20" rot="MR0" align="center">JS220 Binding Post Front Panel
-Rev B
+<text x="28.45" y="20.5" size="3" layer="29" font="vector" ratio="20" distance="40" align="center">Voltage</text>
+<text x="66.55" y="20.5" size="3" layer="29" font="vector" ratio="20" distance="40" align="center">Current</text>
+<text x="47.5" y="20.2" size="1.27" layer="26" font="vector" ratio="20" rot="MR0" align="center">JS220_fp_bp_pcb_revB
+JS220 Binding Post Front Panel, Rev B
 2022 Jetperch LLC</text>
 <dimension x1="0" y1="12.35" x2="95" y2="12.35" x3="47.5" y3="40.64" textsize="1.778" layer="47" dtype="horizontal"/>
-<dimension x1="12.35" y1="0" x2="12.35" y2="24.7" x3="-6.35" y3="12.35" textsize="1.778" layer="47" dtype="vertical"/>
+<dimension x1="12.35" y1="0" x2="12.35" y2="24.7" x3="-17.35" y3="12.35" textsize="1.778" layer="47" dtype="vertical"/>
 <dimension x1="18.925" y1="12.35" x2="37.975" y2="12.35" x3="28.45" y3="-3.81" textsize="1.778" layer="47" dtype="horizontal"/>
 <dimension x1="37.975" y1="12.35" x2="57.025" y2="12.35" x3="47.5" y3="-3.81" textsize="1.778" layer="47" dtype="horizontal"/>
@@
 <wire x1="82.65" y1="24.7" x2="12.35" y2="24.7" width="0" layer="20"/>
 <wire x1="12.35" y1="24.7" x2="0" y2="12.35" width="0" layer="20" curve="90"/>
-<text x="28.45" y="8.968" size="1.5" layer="29" font="vector" ratio="20" align="center">Status</text>
+<text x="28.45" y="8" size="1.5" layer="29" font="vector" ratio="20" align="center">Sensor
+Status</text>
 <hole x="28.45" y="12.5" drill="3.3"/>
 <wire x1="61" y1="8.68" x2="72" y2="8.68" width="0.254" layer="22"/>
@@
 <wire x1="23" y1="8.68" x2="34" y2="8.68" width="0.254" layer="22"/>
 <wire x1="51" y1="7.78" x2="92" y2="7.78" width="0.127" layer="22" style="shortdash"/>
-<dimension x1="47.5" y1="26.6" x2="76.075" y2="12.655" x3="61.7875" y3="36" textsize="1.778" layer="47" dtype="horizontal" precision="3"/>
-<wire x1="21.75" y1="20" x2="20.425" y2="20" width="0.254" layer="29"/>
-<wire x1="20.425" y1="20" x2="19.425" y2="19" width="0.254" layer="29"/>
-<wire x1="19.425" y1="19" x2="19.425" y2="18" width="0.254" layer="29"/>
-<wire x1="35.6" y1="20" x2="36.475" y2="20" width="0.254" layer="29"/>
-<wire x1="36.475" y1="20" x2="37.475" y2="19" width="0.254" layer="29"/>
-<wire x1="37.475" y1="19" x2="37.475" y2="18" width="0.254" layer="29"/>
-<wire x1="59.45" y1="20" x2="58.525" y2="20" width="0.254" layer="29"/>
-<wire x1="58.525" y1="20" x2="57.525" y2="19" width="0.254" layer="29"/>
-<wire x1="57.525" y1="19" x2="57.525" y2="18" width="0.254" layer="29"/>
-<wire x1="73.25" y1="20" x2="74.575" y2="20" width="0.254" layer="29"/>
-<wire x1="74.575" y1="20" x2="75.575" y2="19" width="0.254" layer="29"/>
-<wire x1="75.575" y1="19" x2="75.575" y2="18" width="0.254" layer="29"/>
 <polygon width="0.254" layer="30">
 <vertex x="47.5" y="0"/>
@@
 <wire x1="80" y1="8.68" x2="92" y2="8.68" width="0.254" layer="22"/>
 <text x="47.5" y="2.2" size="1.27" layer="26" font="vector" ratio="20" rot="MR0" align="center">Install J1-J4 with nut on this side</text>
-<text x="28.45" y="17.6022" size="1.27" layer="29" font="vector" ratio="20" distance="25" align="center">±15V</text>
-<text x="47.5" y="3.2512" size="1.27" layer="29" font="vector" ratio="20" distance="25" align="center">Isolated
+<text x="28.45" y="18" size="1.5" layer="29" font="vector" ratio="20" distance="25" align="top-center">±15V</text>
+<text x="47.5" y="4.5" size="1.5" layer="29" font="vector" ratio="20" align="center">Isolated
 ±48V max to USB ground</text>
-<text x="66.55" y="17.6022" size="1.27" layer="29" font="vector" ratio="20" distance="25" align="center">±3A</text>
+<text x="66.55" y="18" size="1.5" layer="29" font="vector" ratio="20" distance="25" align="top-center">±3A</text>
+<text x="12.573" y="-24.892" size="1.778" layer="153">Place all markings on back (including pcb order number).
+Add flammability rating marking on back, such as 94V-0.
+The front-side surface is cosmetic - reject units with scratches and blemishes.</text>
+<text x="18.925" y="20.5" size="3" layer="29" font="vector" ratio="20" distance="40" align="center">-</text>
+<text x="37.975" y="20.5" size="3" layer="29" font="vector" ratio="20" distance="40" align="center">+</text>
+<text x="57.025" y="20.5" size="3" layer="29" font="vector" ratio="20" distance="40" align="center">+</text>
+<text x="76.075" y="20.5" size="3" layer="29" font="vector" ratio="20" distance="40" align="center">-</text>
+<wire x1="64.1" y1="12.35" x2="69" y2="12.35" width="0.8" layer="29"/>
+<wire x1="69" y1="12.35" x2="68" y2="13.35" width="0.8" layer="29"/>
+<wire x1="69" y1="12.35" x2="68" y2="11.35" width="0.8" layer="29"/>
+<wire x1="68" y1="11.35" x2="68" y2="13.35" width="0.8" layer="29"/>
+<text x="66.55" y="7.7" size="1.5" layer="29" font="vector" ratio="20" distance="25" align="top-center">±10A pulse</text>
+<dimension x1="57.025" y1="12.35" x2="76.075" y2="12.35" x3="66.55" y3="-3.81" textsize="1.778" layer="47" dtype="horizontal"/>
+<dimension x1="0" y1="0" x2="0" y2="12.35" x3="-4.35" y3="6.175" textsize="1.778" layer="47" dtype="vertical"/>
+<dimension x1="28.45" y1="0" x2="28.45" y2="12.5" x3="-12.35" y3="6.25" textsize="1.778" layer="47" dtype="vertical"/>
+<text x="-11.2" y="6.1" size="0.9" layer="47" rot="R90" align="center">Sensor Status</text>
+<text x="-2.9" y="6.3" size="0.9" layer="47" rot="R90" align="center">2x holes
+4x connectors</text>
 </plain>
 <attributes>
@@
 <attribute name="POPULATE" value="0" x="87.21" y="3.81" size="1.778" layer="28" rot="MR0" display="off"/>
 </element>
-<element name="H2" library="jetperch" package="HOLE_3.5MM_NORESTRICT" value="HOLE_#6_NORESTRICT" x="3.79" y="12.35" smashed="yes"/>
-<element name="H3" library="jetperch" package="HOLE_3.5MM_NORESTRICT" value="HOLE_#6_NORESTRICT" x="91.21" y="12.35" smashed="yes"/>
+<element name="H1" library="jetperch" package="HOLE_3.5MM_NORESTRICT" value="HOLE_#6_NORESTRICT" x="3.79" y="12.35" smashed="yes">
+<attribute name="POPULATE" value="0" x="3.79" y="12.35" size="1.778" layer="27" display="off"/>
+</element>
+<element name="H2" library="jetperch" package="HOLE_3.5MM_NORESTRICT" value="HOLE_#6_NORESTRICT" x="91.21" y="12.35" smashed="yes">
+<attribute name="POPULATE" value="0" x="91.21" y="12.35" size="1.778" layer="27" display="off"/>
+</element>
 <element name="J2" library="jetperch" package="BINDING_POST_6" value="111-0702-001" x="37.975" y="12.35" smashed="yes">
 <attribute name="MPN" value="111-0702-001" x="37.975" y="12.35" size="1.778" layer="27" display="off"/>
@@
 <contactref element="J1" pad="1"/>
 <contactref element="J5" pad="5"/>
-<wire x1="44.96" y1="6.322" x2="42.829" y2="4.191" width="1.27" layer="16"/>
-<wire x1="42.829" y1="4.191" x2="27.084" y2="4.191" width="1.27" layer="16"/>
-<wire x1="27.084" y1="4.191" x2="18.925" y2="12.35" width="1.27" layer="16"/>
+<wire x1="44.96" y1="6.322" x2="43.21" y2="4.572" width="1.27" layer="16"/>
+<wire x1="43.21" y1="4.572" x2="26.703" y2="4.572" width="1.27" layer="16"/>
+<wire x1="26.703" y1="4.572" x2="18.925" y2="12.35" width="1.27" layer="16"/>
 <wire x1="44.96" y1="8.5165" x2="44.96" y2="6.322" width="1.27" layer="16"/>
 </signal>
@@
 <vertex x="46.99" y="14.732"/>
 <vertex x="46.99" y="19.431"/>
-<vertex x="49.149" y="21.59"/>
-<vertex x="72.898" y="21.59"/>
+<vertex x="49.657" y="22.098"/>
+<vertex x="72.39" y="22.098"/>
 <vertex x="79.121" y="15.367"/>
 <vertex x="79.121" y="9.398"/>
-<vertex x="72.136" y="2.413"/>
-<vertex x="48.895" y="2.413"/>
+<vertex x="72.263" y="2.54"/>
+<vertex x="48.768" y="2.54"/>
 <vertex x="46.99" y="4.318"/>
 <vertex x="46.99" y="7.112"/>
@@
 </signal>
 <signal name="CGND">
-<polygon width="0.254" layer="1" isolate="0.254">
+<polygon width="0.254" layer="1" isolate="0.508">
 <vertex x="12.35" y="24.7"/>
 <vertex x="82.65" y="24.7" curve="-90"/>

Commit message: Final build files.
Fixed fp_binding_posts with corrected connector.
Parts:
- J5: value TSM-105-01-L-SV-A -> TSM-103-01-S-DV-A
Changed lines of the file:
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@@
 </autorouter>
 <elements>
-<element name="J5" library="jetperch" package="CONN_0.1_3X2_MSA" value="TSM-105-01-L-SV-A" x="47.5" y="11.0565" smashed="yes" rot="MR0">
-<attribute name="MPN" value="TSM-105-01-L-SV-A" x="47.5" y="11.0565" size="1.778" layer="28" rot="MR0" display="off"/>
+<element name="J5" library="jetperch" package="CONN_0.1_3X2_MSA" value="TSM-103-01-S-DV-A" x="47.5" y="11.0565" smashed="yes" rot="MR0">
+<attribute name="MPN" value="TSM-103-01-S-DV-A" x="47.5" y="11.0565" size="1.778" layer="28" rot="MR0" display="off"/>
 <attribute name="NAME" x="51.642" y="5.3865" size="0.8128" layer="26" font="vector" ratio="22" rot="MR0"/>
 <attribute name="POPULATE" value="1" x="47.5" y="11.0565" size="1.778" layer="28" rot="MR0" display="off"/>

Commit message: Updated for beta build.
Other:
- board text added: "JS220_fp_bp_pcb_revC JS220 Binding Post Front Panel, Rev C 2022 Jetperch LLC"
- board text removed: "JS220_fp_bp_pcb_revB JS220 Binding Post Front Panel, Rev B 2022 Jetperch LLC"
Changed lines of the file:
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@@
 <text x="28.45" y="20.5" size="3" layer="29" font="vector" ratio="20" distance="40" align="center">Voltage</text>
 <text x="66.55" y="20.5" size="3" layer="29" font="vector" ratio="20" distance="40" align="center">Current</text>
-<text x="47.5" y="20.2" size="1.27" layer="26" font="vector" ratio="20" rot="MR0" align="center">JS220_fp_bp_pcb_revB
-JS220 Binding Post Front Panel, Rev B
+<text x="47.5" y="20.2" size="1.27" layer="26" font="vector" ratio="20" rot="MR0" align="center">JS220_fp_bp_pcb_revC
+JS220 Binding Post Front Panel, Rev C
 2022 Jetperch LLC</text>
 <dimension x1="0" y1="12.35" x2="95" y2="12.35" x3="47.5" y3="40.64" textsize="1.778" layer="47" dtype="horizontal"/>
