File: eagle/fp_safety_banana/js220_fp_sba.brd (EAGLE design)
At the start: 95 x 24.7 mm, 10 parts, among them J1 CT3151V1-0, J2 CT3149-2, J3 CT3151V1-2, J4 CT3151V1-4, J5 TSM-103-01-S-DV-A

Commit message: Added safety banana jack rev B with same connectors as JS110
Parts:
- J1: value CT3151V1-0 -> CT3149-0; device jetperch:CT3151V -> jetperch:CT3149
- J2: device jetperch:CT3151V -> jetperch:CT3149
- J3: value CT3151V1-2 -> CT3149-2; device jetperch:CT3151V -> jetperch:CT3149
- J4: value CT3151V1-4 -> CT3149-4; device jetperch:CT3151V -> jetperch:CT3149
Connections:
- net I+: now also J3.A; no longer J3.1, J3.2, J3.3, J3.4
- net I-: now also J4.A; no longer J4.1, J4.2, J4.3, J4.4
- net V+: now also J2.A; no longer J2.1, J2.2, J2.3, J2.4
- net V-: now also J1.A; no longer J1.1, J1.2, J1.3, J1.4
Routing:
- net V+: track 19.0 -> 7.50 mm
- net V-: track 42.2 -> 31.1 mm
- net I-: track 79.4 -> 70.7 mm
- net I+: track 25.2 -> 16.4 mm
Other:
- board text added: "2024 Jetperch LLC"
- board text added: "JS220_fp_sba_pcb_revB JS220 Safety Banana Jack Front Panel Rev B"
- board text removed: "2023 Jetperch LLC"
- board text removed: "JS220_fp_banana_pcb_revC JS220 Safety Banana Jack Front Panel Rev A"
Changed lines of the file:
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@@
 <drawing>
 <settings>
-<setting alwaysvectorfont="no"/>
+<setting alwaysvectorfont="yes"/>
 <setting verticaltext="up"/>
 </settings>
@@
 <text x="28.45" y="20.5" size="3" layer="29" font="vector" ratio="20" distance="40" align="center">Voltage</text>
 <text x="66.55" y="20.5" size="3" layer="29" font="vector" ratio="20" distance="40" align="center">Current</text>
-<text x="28.45" y="20.2" size="1.27" layer="26" font="vector" ratio="20" rot="MR0" align="center">JS220_fp_banana_pcb_revC
+<text x="28.45" y="20.2" size="1.27" layer="26" font="vector" ratio="20" rot="MR0" align="center">JS220_fp_sba_pcb_revB
 JS220 Safety Banana Jack Front Panel
-Rev A</text>
+Rev B</text>
 <dimension x1="0" y1="12.35" x2="95" y2="12.35" x3="47.5" y3="40.64" textsize="1.778" layer="47" dtype="horizontal"/>
 <dimension x1="12.35" y1="0" x2="12.35" y2="24.7" x3="-17.35" y3="12.35" textsize="1.778" layer="47" dtype="vertical"/>
@@
 <wire x1="49.149" y1="22.225" x2="46.228" y2="19.304" width="0.254" layer="30"/>
 <wire x1="46.228" y1="19.304" x2="46.228" y2="16.891" width="0.254" layer="30"/>
-<text x="28.45" y="2.5" size="1.27" layer="26" font="vector" ratio="20" rot="MR0" align="center">2023 Jetperch LLC</text>
+<text x="28.45" y="2.5" size="1.27" layer="26" font="vector" ratio="20" rot="MR0" align="center">2024 Jetperch LLC</text>
 <wire x1="46" y1="4" x2="45" y2="3" width="0.254" layer="30"/>
 <wire x1="45" y1="3" x2="36.7" y2="3" width="0.254" layer="30"/>
@@
 <attribute name="POPULATE" value="1" x="47.5" y="11.0565" size="1.778" layer="28" rot="MR0" display="off"/>
 </element>
-<element name="J1" library="jetperch" package="CT3151V" value="CT3151V1-0" x="18.925" y="12.35" smashed="yes">
+<element name="J1" library="jetperch" package="CT3149" value="CT3149-0" x="18.925" y="12.35" smashed="yes">
 <attribute name="MPN" value="CT3151V1-0" x="18.925" y="12.35" size="1.778" layer="27" display="off"/>
 <attribute name="POPULATE" value="1" x="18.925" y="12.35" size="1.778" layer="27" display="off"/>
 </element>
-<element name="J3" library="jetperch" package="CT3151V" value="CT3151V1-2" x="57.025" y="12.35" smashed="yes">
+<element name="J3" library="jetperch" package="CT3149" value="CT3149-2" x="57.025" y="12.35" smashed="yes">
 <attribute name="MPN" value="CT3151V1-2" x="57.025" y="12.35" size="1.778" layer="27" display="off"/>
 <attribute name="POPULATE" value="1" x="57.025" y="12.35" size="1.778" layer="27" display="off"/>
 </element>
-<element name="J4" library="jetperch" package="CT3151V" value="CT3151V1-4" x="76.075" y="12.35" smashed="yes">
+<element name="J4" library="jetperch" package="CT3149" value="CT3149-4" x="76.075" y="12.35" smashed="yes">
 <attribute name="MPN" value="CT3151V1-4" x="76.075" y="12.35" size="1.778" layer="27" display="off"/>
 <attribute name="POPULATE" value="1" x="76.075" y="12.35" size="1.778" layer="27" display="off"/>
@@
 <attribute name="POPULATE" value="0" x="91.21" y="12.35" size="1.778" layer="27" display="off"/>
 </element>
-<element name="J2" library="jetperch" package="CT3151V" value="CT3149-2" x="37.975" y="12.35" smashed="yes">
+<element name="J2" library="jetperch" package="CT3149" value="CT3149-2" x="37.975" y="12.35" smashed="yes">
 <attribute name="MPN" value="CT3151V1-2" x="37.975" y="12.35" size="1.778" layer="27" display="off"/>
 <attribute name="POPULATE" value="1" x="37.975" y="12.35" size="1.778" layer="27" display="off"/>
@@
 <signals>
 <signal name="I+">
-<contactref element="J3" pad="1"/>
+<contactref element="J3" pad="A"/>
 <contactref element="J5" pad="1"/>
 <contactref element="J5" pad="2"/>
@@
 <vertex x="49.657" y="9.271"/>
 </polygon>
-<contactref element="J3" pad="2"/>
-<contactref element="J3" pad="3"/>
-<contactref element="J3" pad="4"/>
-<wire x1="53.1915" y1="8.5165" x2="55.34" y2="10.665" width="0.254" layer="16"/>
+<wire x1="53.1915" y1="8.5165" x2="57.025" y2="12.35" width="0.254" layer="16"/>
 <wire x1="50.04" y1="13.5965" x2="50.4785" y2="14.035" width="0.254" layer="16"/>
 <wire x1="50.4785" y1="14.035" x2="55.34" y2="14.035" width="0.254" layer="16"/>
-<wire x1="55.34" y1="14.035" x2="58.71" y2="14.035" width="0.254" layer="16"/>
-<wire x1="58.71" y1="14.035" x2="58.71" y2="10.665" width="0.254" layer="16"/>
-<wire x1="58.71" y1="10.665" x2="55.34" y2="10.665" width="0.254" layer="16"/>
-<wire x1="55.34" y1="10.665" x2="55.34" y2="14.035" width="0.254" layer="16"/>
+<wire x1="57.025" y1="12.35" x2="55.34" y2="14.035" width="0.254" layer="16"/>
 </signal>
 <signal name="V-">
-<contactref element="J1" pad="1"/>
+<contactref element="J1" pad="A"/>
 <contactref element="J5" pad="5"/>
-<contactref element="J1" pad="2"/>
-<contactref element="J1" pad="3"/>
-<contactref element="J1" pad="4"/>
-<wire x1="17.24" y1="14.035" x2="17.24" y2="10.665" width="1" layer="16"/>
-<wire x1="17.24" y1="10.665" x2="20.61" y2="10.665" width="1" layer="16"/>
-<wire x1="20.61" y1="10.665" x2="20.61" y2="14.035" width="1" layer="16"/>
-<wire x1="20.61" y1="14.035" x2="17.24" y2="14.035" width="1" layer="16"/>
-<wire x1="20.61" y1="10.665" x2="26.275" y2="5" width="1" layer="16"/>
 <wire x1="44.96" y1="7.5165" x2="44.96" y2="8.5165" width="1" layer="16"/>
 <wire x1="44.96" y1="7.5165" x2="42.4435" y2="5" width="1" layer="16"/>
 <wire x1="26.275" y1="5" x2="42.4435" y2="5" width="1" layer="16"/>
+<wire x1="18.925" y1="12.35" x2="26.275" y2="5" width="1" layer="16"/>
 </signal>
 <signal name="I-">
-<contactref element="J4" pad="1"/>
+<contactref element="J4" pad="A"/>
 <contactref element="J5" pad="4"/>
 <contactref element="J5" pad="3"/>
@@
 <wire x1="47.5" y1="5.5" x2="48" y2="5" width="0.254" layer="16"/>
 <wire x1="48" y1="5" x2="68.725" y2="5" width="0.254" layer="16"/>
-<wire x1="68.725" y1="5" x2="74.39" y2="10.665" width="0.254" layer="16"/>
+<wire x1="68.725" y1="5" x2="76.075" y2="12.35" width="0.254" layer="16"/>
 <wire x1="47.5" y1="13.5965" x2="47.5" y2="17.5" width="0.254" layer="16"/>
 <wire x1="49" y1="19" x2="47.5" y2="17.5" width="0.254" layer="16"/>
@@
 <vertex x="47.879" y="14.732"/>
 </polygon>
-<contactref element="J4" pad="2"/>
-<contactref element="J4" pad="3"/>
-<contactref element="J4" pad="4"/>
 <wire x1="66" y1="19" x2="49" y2="19" width="0.254" layer="16"/>
 <wire x1="66" y1="19" x2="70.965" y2="14.035" width="0.254" layer="16"/>
 <wire x1="70.965" y1="14.035" x2="74.39" y2="14.035" width="0.254" layer="16"/>
-<wire x1="74.39" y1="14.035" x2="77.76" y2="14.035" width="0.254" layer="16"/>
-<wire x1="77.76" y1="14.035" x2="77.76" y2="10.665" width="0.254" layer="16"/>
-<wire x1="77.76" y1="10.665" x2="74.39" y2="10.665" width="0.254" layer="16"/>
-<wire x1="74.39" y1="10.665" x2="74.39" y2="14.035" width="0.254" layer="16"/>
+<wire x1="76.075" y1="12.35" x2="74.39" y2="14.035" width="0.254" layer="16"/>
 </signal>
 <signal name="CGND">
@@
 <signal name="V+">
 <contactref element="J5" pad="6"/>
-<contactref element="J2" pad="1"/>
-<contactref element="J2" pad="2"/>
-<contactref element="J2" pad="3"/>
-<contactref element="J2" pad="4"/>
-<wire x1="44.96" y1="13.5965" x2="40.0985" y2="13.5965" width="1" layer="16"/>
-<wire x1="40.0985" y1="13.5965" x2="39.66" y2="14.035" width="1" layer="16"/>
-<wire x1="39.66" y1="14.035" x2="36.29" y2="14.035" width="1" layer="16"/>
-<wire x1="36.29" y1="14.035" x2="36.29" y2="10.665" width="1" layer="16"/>
-<wire x1="36.29" y1="10.665" x2="39.66" y2="10.665" width="1" layer="16"/>
-<wire x1="39.66" y1="10.665" x2="39.66" y2="14.035" width="1" layer="16"/>
+<contactref element="J2" pad="A"/>
+<wire x1="37.975" y1="12.35" x2="39.2215" y2="13.5965" width="1" layer="16"/>
+<wire x1="39.2215" y1="13.5965" x2="44.96" y2="13.5965" width="1" layer="16"/>
 </signal>
 </signals>
