File: eagle/fp_safety_banana/js220_fp_sba.sch (EAGLE design)
At the start: 10 parts, among them J1 CT3151V1-0, J2 CT3149-2, J3 CT3151V1-2, J4 CT3151V1-4, J5 TSM-103-01-S-DV-A

Commit message: Renamed js220_fp_banana to js220_fp_sba
Changed lines of the file:
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@@
 <attribute name="POPULATE" value="1"/>
 </part>
-<part name="PCB1" library="jetperch" deviceset="PCB" device="" value="JS220_fp_banana_pcb_revA">
+<part name="PCB1" library="jetperch" deviceset="PCB" device="" value="JS220_fp_sba_pcb_revA">
 <attribute name="POPULATE" value="1"/>
 </part>

Commit message: Added safety banana jack rev B with same connectors as JS110
Parts:
- J1: value CT3151V1-0 -> CT3149-0; device jetperch:BANANA-JACK_CT3151V -> jetperch:BANANA-JACK_CT3149
- J2: device jetperch:BANANA-JACK_CT3151V -> jetperch:BANANA-JACK_CT3149
- J3: value CT3151V1-2 -> CT3149-2; device jetperch:BANANA-JACK_CT3151V -> jetperch:BANANA-JACK_CT3149
- J4: value CT3151V1-4 -> CT3149-4; device jetperch:BANANA-JACK_CT3151V -> jetperch:BANANA-JACK_CT3149
Other:
- note added: "B"
- note removed: "A"
Changed lines of the file:
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@@
 <grid distance="0.1" unitdist="inch" unit="inch" style="lines" multiple="1" display="no" altdistance="0.01" altunitdist="inch" altunit="inch"/>
 <layers>
-<layer number="1" name="Top" color="4" fill="1" visible="no" active="no"/>
-<layer number="2" name="Route2" color="1" fill="3" visible="no" active="no"/>
-<layer number="3" name="Route3" color="4" fill="3" visible="no" active="no"/>
-<layer number="4" name="Route4" color="1" fill="4" visible="no" active="no"/>
-<layer number="5" name="Route5" color="4" fill="4" visible="no" active="no"/>
-<layer number="6" name="Route6" color="1" fill="8" visible="no" active="no"/>
-<layer number="7" name="Route7" color="4" fill="8" visible="no" active="no"/>
-<layer number="8" name="Route8" color="1" fill="2" visible="no" active="no"/>
-<layer number="9" name="Route9" color="4" fill="2" visible="no" active="no"/>
-<layer number="10" name="Route10" color="1" fill="7" visible="no" active="no"/>
-<layer number="11" name="Route11" color="4" fill="7" visible="no" active="no"/>
-<layer number="12" name="Route12" color="1" fill="5" visible="no" active="no"/>
-<layer number="13" name="Route13" color="4" fill="5" visible="no" active="no"/>
-<layer number="14" name="Route14" color="1" fill="6" visible="no" active="no"/>
-<layer number="15" name="Route15" color="4" fill="6" visible="no" active="no"/>
-<layer number="16" name="Bottom" color="1" fill="1" visible="no" active="no"/>
-<layer number="17" name="Pads" color="2" fill="1" visible="no" active="no"/>
-<layer number="18" name="Vias" color="2" fill="1" visible="no" active="no"/>
-<layer number="19" name="Unrouted" color="6" fill="1" visible="no" active="no"/>
-<layer number="20" name="Dimension" color="24" fill="1" visible="no" active="no"/>
-<layer number="21" name="tPlace" color="7" fill="1" visible="no" active="no"/>
-<layer number="22" name="bPlace" color="7" fill="1" visible="no" active="no"/>
-<layer number="23" name="tOrigins" color="15" fill="1" visible="no" active="no"/>
-<layer number="24" name="bOrigins" color="15" fill="1" visible="no" active="no"/>
-<layer number="25" name="tNames" color="7" fill="1" visible="no" active="no"/>
-<layer number="26" name="bNames" color="7" fill="1" visible="no" active="no"/>
-<layer number="27" name="tValues" color="7" fill="1" visible="no" active="no"/>
-<layer number="28" name="bValues" color="7" fill="1" visible="no" active="no"/>
+<layer number="1" name="Top" color="4" fill="1" visible="yes" active="no"/>
+<layer number="2" name="Route2" color="1" fill="3" visible="yes" active="no"/>
+<layer number="3" name="Route3" color="4" fill="3" visible="yes" active="no"/>
+<layer number="4" name="Route4" color="1" fill="4" visible="yes" active="no"/>
+<layer number="5" name="Route5" color="4" fill="4" visible="yes" active="no"/>
+<layer number="6" name="Route6" color="1" fill="8" visible="yes" active="no"/>
+<layer number="7" name="Route7" color="4" fill="8" visible="yes" active="no"/>
+<layer number="8" name="Route8" color="1" fill="2" visible="yes" active="no"/>
+<layer number="9" name="Route9" color="4" fill="2" visible="yes" active="no"/>
+<layer number="10" name="Route10" color="1" fill="7" visible="yes" active="no"/>
+<layer number="11" name="Route11" color="4" fill="7" visible="yes" active="no"/>
+<layer number="12" name="Route12" color="1" fill="5" visible="yes" active="no"/>
+<layer number="13" name="Route13" color="4" fill="5" visible="yes" active="no"/>
+<layer number="14" name="Route14" color="1" fill="6" visible="yes" active="no"/>
+<layer number="15" name="Route15" color="4" fill="6" visible="yes" active="no"/>
+<layer number="16" name="Bottom" color="1" fill="1" visible="yes" active="no"/>
+<layer number="17" name="Pads" color="2" fill="1" visible="yes" active="no"/>
+<layer number="18" name="Vias" color="2" fill="1" visible="yes" active="no"/>
+<layer number="19" name="Unrouted" color="6" fill="1" visible="yes" active="no"/>
+<layer number="20" name="Dimension" color="24" fill="1" visible="yes" active="no"/>
+<layer number="21" name="tPlace" color="7" fill="1" visible="yes" active="no"/>
+<layer number="22" name="bPlace" color="7" fill="1" visible="yes" active="no"/>
+<layer number="23" name="tOrigins" color="15" fill="1" visible="yes" active="no"/>
+<layer number="24" name="bOrigins" color="15" fill="1" visible="yes" active="no"/>
+<layer number="25" name="tNames" color="7" fill="1" visible="yes" active="no"/>
+<layer number="26" name="bNames" color="7" fill="1" visible="yes" active="no"/>
+<layer number="27" name="tValues" color="7" fill="1" visible="yes" active="no"/>
+<layer number="28" name="bValues" color="7" fill="1" visible="yes" active="no"/>
 <layer number="29" name="tStop" color="7" fill="3" visible="no" active="no"/>
 <layer number="30" name="bStop" color="7" fill="6" visible="no" active="no"/>
@@
 <layer number="35" name="tGlue" color="7" fill="4" visible="no" active="no"/>
 <layer number="36" name="bGlue" color="7" fill="5" visible="no" active="no"/>
-<layer number="37" name="tTest" color="7" fill="1" visible="no" active="no"/>
-<layer number="38" name="bTest" color="7" fill="1" visible="no" active="no"/>
+<layer number="37" name="tTest" color="7" fill="1" visible="yes" active="no"/>
+<layer number="38" name="bTest" color="7" fill="1" visible="yes" active="no"/>
 <layer number="39" name="tKeepout" color="4" fill="11" visible="no" active="no"/>
 <layer number="40" name="bKeepout" color="1" fill="11" visible="no" active="no"/>
@@
 <layer number="44" name="Drills" color="7" fill="1" visible="no" active="no"/>
 <layer number="45" name="Holes" color="7" fill="1" visible="no" active="no"/>
-<layer number="46" name="Milling" color="3" fill="1" visible="no" active="no"/>
-<layer number="47" name="Measures" color="7" fill="1" visible="no" active="no"/>
-<layer number="48" name="Document" color="7" fill="1" visible="no" active="no"/>
-<layer number="49" name="Reference" color="7" fill="1" visible="no" active="no"/>
-<layer number="50" name="dxf" color="7" fill="1" visible="no" active="no"/>
-<layer number="51" name="tDocu" color="7" fill="1" visible="no" active="no"/>
-<layer number="52" name="bDocu" color="7" fill="1" visible="no" active="no"/>
-<layer number="53" name="tGND_GNDA" color="7" fill="9" visible="no" active="no"/>
-<layer number="54" name="bGND_GNDA" color="1" fill="9" visible="no" active="no"/>
-<layer number="56" name="wert" color="7" fill="1" visible="no" active="no"/>
-<layer number="57" name="tCAD" color="7" fill="1" visible="no" active="no"/>
-<layer number="59" name="tCarbon" color="7" fill="1" visible="no" active="no"/>
-<layer number="60" name="bCarbon" color="7" fill="1" visible="no" active="no"/>
+<layer number="46" name="Milling" color="3" fill="1" visible="yes" active="no"/>
+<layer number="47" name="Measures" color="7" fill="1" visible="yes" active="no"/>
+<layer number="48" name="Document" color="7" fill="1" visible="yes" active="no"/>
+<layer number="49" name="Reference" color="7" fill="1" visible="yes" active="no"/>
+<layer number="50" name="dxf" color="7" fill="1" visible="yes" active="no"/>
+<layer number="51" name="tDocu" color="7" fill="1" visible="yes" active="no"/>
+<layer number="52" name="bDocu" color="7" fill="1" visible="yes" active="no"/>
+<layer number="53" name="tGND_GNDA" color="7" fill="9" visible="yes" active="no"/>
+<layer number="54" name="bGND_GNDA" color="1" fill="9" visible="yes" active="no"/>
+<layer number="56" name="wert" color="7" fill="1" visible="yes" active="no"/>
+<layer number="57" name="tCAD" color="7" fill="1" visible="yes" active="no"/>
+<layer number="59" name="tCarbon" color="7" fill="1" visible="yes" active="no"/>
+<layer number="60" name="bCarbon" color="7" fill="1" visible="yes" active="no"/>
 <layer number="88" name="SimResults" color="9" fill="1" visible="yes" active="yes"/>
 <layer number="89" name="SimProbes" color="9" fill="1" visible="yes" active="yes"/>
@@
 <attribute name="POPULATE" value="1"/>
 </part>
-<part name="J1" library="jetperch" deviceset="BANANA-JACK" device="_CT3151V" value="CT3151V1-0">
+<part name="J1" library="jetperch" deviceset="BANANA-JACK" device="_CT3149" value="CT3149-0">
 <attribute name="MPN" value="CT3151V1-0"/>
 <attribute name="POPULATE" value="1"/>
 </part>
-<part name="J3" library="jetperch" deviceset="BANANA-JACK" device="_CT3151V" value="CT3151V1-2">
+<part name="J3" library="jetperch" deviceset="BANANA-JACK" device="_CT3149" value="CT3149-2">
 <attribute name="MPN" value="CT3151V1-2"/>
 <attribute name="POPULATE" value="1"/>
 </part>
-<part name="J4" library="jetperch" deviceset="BANANA-JACK" device="_CT3151V" value="CT3151V1-4">
+<part name="J4" library="jetperch" deviceset="BANANA-JACK" device="_CT3149" value="CT3149-4">
 <attribute name="MPN" value="CT3151V1-4"/>
 <attribute name="POPULATE" value="1"/>
@@
 <attribute name="POPULATE" value="0"/>
 </part>
-<part name="J2" library="jetperch" deviceset="BANANA-JACK" device="_CT3151V" value="CT3149-2">
+<part name="J2" library="jetperch" deviceset="BANANA-JACK" device="_CT3149" value="CT3149-2">
 <attribute name="MPN" value="CT3151V1-2"/>
 <attribute name="POPULATE" value="1"/>
 </part>
-<part name="PCB1" library="jetperch" deviceset="PCB" device="" value="JS220_fp_sba_pcb_revA">
+<part name="PCB1" library="jetperch" deviceset="PCB" device="" value="JS220_fp_sba_pcb_revB">
 <attribute name="POPULATE" value="1"/>
 </part>
@@
 <plain>
 <text x="177.8" y="26.162" size="5.08" layer="97">Front Panel - Banana Jack</text>
-<text x="266.7" y="6.35" size="3.175" layer="97">A</text>
+<text x="266.7" y="6.35" size="3.175" layer="97">B</text>
 <text x="144.78" y="198.12" size="2.54" layer="97" align="center">+            -</text>
 <text x="144.78" y="203.2" size="2.54" layer="97" align="center">AMMETER</text>

Commit message: Added JS220 Safety Banana Jack front panel.
Fixed connector part numbers for BOM.
Parts:
- J1: MPN CT3151V1-0 -> (none)
- J2, J3: MPN CT3151V1-2 -> (none)
- J4: MPN CT3151V1-4 -> (none)
